File: puppet_pcb/puppet_pcb/puppet_pcb.kicad_pcb (KiCad board)
At the start: 2 copper layers, 134 x 94 mm, 52 parts, among them IC1 TEENSY_4.1, J1 CAN, J2 +5V, J3 +12V, J4 M1, J5 M2, J6 M3, J7 M4, J8 Conn_02x20_Odd_Even_MountingP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, U1 MCP2562-E_SN, U10 TB67H420FTG Dual/Single Motor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, U2 MCP2515-I_SO, U3 MCP2562-E_SN, U4 MCP2515-I_SO, U5 ATmega2560-16A, U6 ATmega2560-16A, U7 AVR ISP 6b adapter, U8 AVR ISP 6b adapter, U9 TB67H420FTG Dual/Single Motor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, Y1 16MHz, Y2 16MHz, Y3 16MHz, Y4 16MHz

Commit message: pcb changes
Parts:
- moved R5 2.28 mm to (189.5, 104.5), turned to 90 degrees
Connections:
- C15 pad 2: Net-(IC1-+5V) -> Net-(IC1-VIN_(3.6_TO_5.5_VOLTS))
- C16 pad 2: Net-(IC1-+5V) -> Net-(IC1-VIN_(3.6_TO_5.5_VOLTS))
- C17 pad 2: Net-(IC1-+5V) -> Net-(IC1-VIN_(3.6_TO_5.5_VOLTS))
- C18 pad 2: Net-(IC1-+5V) -> Net-(IC1-VIN_(3.6_TO_5.5_VOLTS))
- C19 pad 2: Net-(IC1-+5V) -> Net-(IC1-VIN_(3.6_TO_5.5_VOLTS))
- C20 pad 2: Net-(IC1-+5V) -> Net-(IC1-VIN_(3.6_TO_5.5_VOLTS))
- C3 pad 1: Net-(IC1-+5V) -> Net-(IC1-VIN_(3.6_TO_5.5_VOLTS))
- C4 pad 2: Net-(IC1-+5V) -> Net-(IC1-VIN_(3.6_TO_5.5_VOLTS))
- C5 pad 2: Net-(IC1-+5V) -> Net-(IC1-VIN_(3.6_TO_5.5_VOLTS))
- C6 pad 1: Net-(IC1-+5V) -> Net-(IC1-VIN_(3.6_TO_5.5_VOLTS))
- IC1 pad 52: Net-(IC1-+5V) -> unconnected-(IC1-+5V-Pad52)
- IC1 pad 55: unconnected-(IC1-VIN_(3.6_TO_5.5_VOLTS)-Pad55) -> Net-(IC1-VIN_(3.6_TO_5.5_VOLTS))
- J2 pad 1: Net-(IC1-+5V) -> Net-(IC1-VIN_(3.6_TO_5.5_VOLTS))
- R1 pad 1: Net-(IC1-+5V) -> Net-(IC1-VIN_(3.6_TO_5.5_VOLTS))
- R6 pad 2: Net-(IC1-+5V) -> Net-(IC1-VIN_(3.6_TO_5.5_VOLTS))
- R7 pad 1: Net-(IC1-+5V) -> Net-(IC1-VIN_(3.6_TO_5.5_VOLTS))
- R8 pad 1: Net-(IC1-+5V) -> Net-(IC1-VIN_(3.6_TO_5.5_VOLTS))
- U1 pad 3: Net-(IC1-+5V) -> Net-(IC1-VIN_(3.6_TO_5.5_VOLTS))
- U1 pad 5: Net-(IC1-+5V) -> Net-(IC1-VIN_(3.6_TO_5.5_VOLTS))
- U2 pad 18: Net-(IC1-+5V) -> Net-(IC1-VIN_(3.6_TO_5.5_VOLTS))
- U3 pad 3: Net-(IC1-+5V) -> Net-(IC1-VIN_(3.6_TO_5.5_VOLTS))
- U3 pad 5: Net-(IC1-+5V) -> Net-(IC1-VIN_(3.6_TO_5.5_VOLTS))
- U4 pad 18: Net-(IC1-+5V) -> Net-(IC1-VIN_(3.6_TO_5.5_VOLTS))
- U5 pad 10: Net-(IC1-+5V) -> Net-(IC1-VIN_(3.6_TO_5.5_VOLTS))
- U5 pad 100: Net-(IC1-+5V) -> Net-(IC1-VIN_(3.6_TO_5.5_VOLTS))
- U5 pad 31: Net-(IC1-+5V) -> Net-(IC1-VIN_(3.6_TO_5.5_VOLTS))
- U5 pad 61: Net-(IC1-+5V) -> Net-(IC1-VIN_(3.6_TO_5.5_VOLTS))
- U5 pad 80: Net-(IC1-+5V) -> Net-(IC1-VIN_(3.6_TO_5.5_VOLTS))
- U6 pad 10: Net-(IC1-+5V) -> Net-(IC1-VIN_(3.6_TO_5.5_VOLTS))
- U6 pad 100: Net-(IC1-+5V) -> Net-(IC1-VIN_(3.6_TO_5.5_VOLTS))
- U6 pad 31: Net-(IC1-+5V) -> Net-(IC1-VIN_(3.6_TO_5.5_VOLTS))
- U6 pad 61: Net-(IC1-+5V) -> Net-(IC1-VIN_(3.6_TO_5.5_VOLTS))
- U6 pad 80: Net-(IC1-+5V) -> Net-(IC1-VIN_(3.6_TO_5.5_VOLTS))
- U7 pad 4: Net-(IC1-+5V) -> Net-(IC1-VIN_(3.6_TO_5.5_VOLTS))
- U8 pad 4: Net-(IC1-+5V) -> Net-(IC1-VIN_(3.6_TO_5.5_VOLTS))
Routing:
- net Net-(IC1-VIN_(3.6_TO_5.5_VOLTS)): track 0.00 -> 462.7 mm, vias 0 -> 10
- net Net-(IC1-+5V): track 461.9 -> 0.00 mm, vias 8 -> 0
- net Net-(IC1-A16): track 36.6 -> 90.0 mm, vias 0 -> 2
- net Net-(IC1-A15): track 35.9 -> 86.6 mm, vias 0 -> 1
- net Net-(IC1-A17): track 46.4 -> 95.6 mm, vias 0 -> 1
- net Net-(J8-Pin_37): track 63.1 -> 94.1 mm
- net Net-(IC1-A12): track 87.1 -> 115.4 mm, vias 0 -> 2
- net Net-(J8-Pin_36): track 31.2 -> 55.7 mm
- net Net-(D1-A2): track 633.2 -> 653.1 mm, vias 9 -> 10
- net Net-(U5-~{RESET}): track 73.5 -> 82.4 mm
- net Net-(J8-Pin_7): track 43.0 -> 50.3 mm
- net Net-(IC1-A5): track 51.6 -> 57.3 mm
- net Net-(IC1-A4): track 57.5 -> 62.8 mm
- net Net-(U6-~{RESET}): track 80.7 -> 85.7 mm
- net Net-(J8-Pin_5): track 48.7 -> 44.9 mm
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