File: puppet_pcb/puppet_pcb/puppet_pcb.kicad_sch (KiCad schematic)
At the start: 36 parts, among them IC1 TEENSY_4.1, J1 CAN, J10 Conn_PIC_ICSP_ICD, J2 +5V, J3 +12V, J4 CAN, J5 CAN, J6 CAN, J7 CAN, J8 Conn_02x20_Odd_Even_MountingP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, J9 Conn_PIC_ICSP_ICD, U1 MCP2515_18L_SOIC, U10 TB67H420FTG Dual/Single Motor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, U2 MCP2562_SOIC, U3 ATmega2560-16A, U4 MCP2515_18L_SOIC, U5 MCP2562_SOIC, U6 ATmega2560-16A, U7 CAN_H, U8 CAN_L, U9 TB67H420FTG Dual/Single Motor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, Y1 16MHz, Y2 16MHz

Commit message: pcb done
Parts:
- removed J10, J9: Conn_PIC_ICSP_ICD, symbol Connector:Conn_PIC_ICSP_ICD
- removed R4: 10kΩ, symbol Device:R
- removed U1, U4: MCP2515_18L_SOIC, symbol custom:MCP2515_18lead_SOIC
- removed U2, U5: MCP2562_SOIC, symbol custom:MCP2562_SOIC
- removed U7: CAN_H, symbol custom:CAN_H
- removed U8: CAN_L, symbol custom:CAN_L
- added C10, C11, C12, C9: 22pF, Capacitor_SMD:C_0805_2012Metric, symbol Device:C
- added C13, C14, C15, C16, C17, C18, C19, C20: 100nF, Capacitor_SMD:C_0805_2012Metric, symbol Device:C
- added R3, R5: 1kΩ, Resistor_SMD:R_0805_2012Metric, symbol Device:R
- added R6, R7, R8: 10kΩ, Resistor_SMD:R_0805_2012Metric, symbol Device:R
- added U1, U3: MCP2562-E_SN, custom:MCP2562-E_SN, symbol custom:MCP2562-E_SN
- added U2, U4: MCP2515-I_SO, custom:MCP2515-I_SO, symbol custom:MCP2515-I_SO
- added U7, U8: AVR ISP 6b adapter, custom:Adafruit 6_isp avr adapter, symbol custom:Adapter_AVR_ISP
- added Y3, Y4: 16MHz, custom:perçant_quartz, symbol Device:Crystal
- C1, C2, C3, C4, C5, C6, C7, C8: footprint (none) -> Capacitor_SMD:C_0805_2012Metric
- D1, D2: footprint (none) -> Diode_SMD:Nexperia_DSN0603-2_0.6x0.3mm_P0.4mm
- IC1: footprint TEENSY_4.1:TEENSY41 -> custom:TEENSY_4.1
- J1, J2, J3: footprint (none) -> TerminalBlock:TerminalBlock_MaiXu_MX126-5.0-02P_1x02_P5.00mm
- J4: value CAN -> M1; footprint (none) -> TerminalBlock:TerminalBlock_MaiXu_MX126-5.0-02P_1x02_P5.00mm
- J5: value CAN -> M2; footprint (none) -> TerminalBlock:TerminalBlock_MaiXu_MX126-5.0-02P_1x02_P5.00mm
- J6: value CAN -> M3; footprint (none) -> TerminalBlock:TerminalBlock_MaiXu_MX126-5.0-02P_1x02_P5.00mm
- J7: value CAN -> M4; footprint (none) -> TerminalBlock:TerminalBlock_MaiXu_MX126-5.0-02P_1x02_P5.00mm
- J8: footprint (none) -> Connector_IDC:IDC-Header_2x20_P2.54mm_Vertical
- R1, R2: footprint (none) -> Resistor_SMD:R_0805_2012Metric
- U10, U9: footprint (none) -> custom:TB67H420FTG Dual_Single Motor
- Y1, Y2: footprint (none) -> custom:perçant_quartz
- renumbered U3 to U5
Connections:
- net at C3.2, C4.1, C5.1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: now also U10.2 (GND), U9.2 (GND), C13.2, C14.2, C15.1, C16.1, C17.1, C18.1, C19.1, C20.1, U1.2 (VSS), U1.8 (STBY), U2.9 (VSS), U3.2 (VSS), U3.8 (STBY), U4.9 (VSS), U7.6 (GND), U8.6 (GND); no longer U10. (A+), U9. (A+)
- net at IC1.22 (A8): now also U9.11 (PWMB); no longer U9. (A+)
- net at IC1.23 (A9): now also U9.14 (PWMA); no longer U9. (A+)
- net at IC1.24 (A10): now also U9.16 (INA1); no longer U9. (A+)
- net at IC1.25 (A11): now also U9.15 (INA2); no longer U9. (A+)
- net at IC1.26 (A12): now also U9.13 (INB1); no longer U9. (A+)
- net at IC1.27 (A13): now also U9.12 (INB2); no longer U9. (A+)
- net at J5.1 (Pin_1): now also U9.6 (A-); no longer U9. (A+)
- net at J5.2 (Pin_2): now also U9.5 (B-); no longer U9. (A+)
- net at J4.1 (Pin_1): now also U9.3 (GND); no longer U9. (A+)
- net at J4.2 (Pin_2): now also U9.4 (B+); no longer U9. (A+)
- net at IC1.14 (A0): now also U10.11 (PWMB); no longer U10. (A+)
- net at IC1.15 (A1): now also U10.14 (PWMA); no longer U10. (A+)
- net at IC1.18 (A4): now also U10.12 (INB2); no longer U10. (A+)
- net at IC1.19 (A5): now also U10.13 (INB1); no longer U10. (A+)
- net at IC1.20 (A6): now also U10.15 (INA2); no longer U10. (A+)
- net at IC1.21 (A7): now also U10.16 (INA1); no longer U10. (A+)
- net at J7.1 (Pin_1): now also U10.6 (A-); no longer U10. (A+)
- net at J7.2 (Pin_2): now also U10.5 (B-); no longer U10. (A+)
- net at J6.1 (Pin_1): now also U10.3 (GND); no longer U10. (A+)
- net at J6.2 (Pin_2): now also U10.4 (B+); no longer U10. (A+)
- net at C3.1, C4.2, C5.2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: now also C15.2, C16.2, C17.2, C18.2, C19.2, C20.2, R6.2, R7.1, R8.1, U1.3 (VDD), U1.5 (VIO), U2.18 (VDD), U3.3 (VDD), U3.5 (VIO), U4.18 (VDD), U7.4 (VCC), U8.4 (VCC)
- net at D1.1 (A1), J1.2 (Pin_2), R2.1: now also U1.7 (CANH), U3.7 (CANH)
- net at U6.19 (PB0): now also U4.16 (~{CS})
- net at U6.20 (PB1): now also U4.13 (SCK), U8.2 (SCK)
- net at U6.21 (PB2): now also U4.14 (SI), U8.5 (MOSI)
- net at U6.22 (PB3): now also U4.15 (SO), U8.1 (MISO)
- net at U6.30 (~{RESET}): now also R5.2, R7.2, U8.3 (RST); no longer J8.36 (Pin_36)
- net at U6.33 (XTAL2): now also C10.1, Y3.2
- net at U6.34 (XTAL1): now also C9.1, Y3.1
- net at U6.6 (PE4): now also U4.12 (~{INT})
- net at U6.98 (AREF): now also C14.1
- net at D2.1 (A1), J1.1 (Pin_1), R2.2: now also U1.6 (CANL), U3.6 (CANL)
- net at C7.1, Y2.1: now also U4.8 (OSC1)
- net at C8.1, Y2.2: now also U4.7 (OSC2)
- net at U5.30 (~{RESET}): now also R3.1, R6.1, U7.3 (RST); no longer J8.37 (Pin_37)
- net at U5.6 (PE4): now also U2.12 (~{INT})
- net at U5.20 (PB1): now also U2.13 (SCK), U7.2 (SCK)
- net at U5.21 (PB2): now also U2.14 (SI), U7.5 (MOSI)
- net at U5.22 (PB3): now also U2.15 (SO), U7.1 (MISO)
- net at U5.19 (PB0): now also U2.16 (~{CS})
- net at R1.2: now also U2.17 (~{RESET})
- net at C1.1, Y1.1: now also U2.8 (OSC1)
- net at C2.1, Y1.2: now also U2.7 (OSC2)
- net at U5.33 (XTAL2): now also C11.1, Y4.2
- net at U5.34 (XTAL1): now also C12.1, Y4.1
- net at U5.98 (AREF): now also C13.1
- new net: J3.1 (Pin_1), U10.1 (VIN), U9.1 (VIN)
- new net: C10.2, C9.2
- new net: U1.1 (TXD), U2.2 (RXCAN)
- new net: U1.4 (RXD), U2.1 (TXCAN)
- new net: C11.2, C12.2
- new net: J8.37 (Pin_37), R3.2
- new net: U3.1 (TXD), U4.2 (RXCAN)
- new net: U3.4 (RXD), U4.1 (TXCAN)
- new net: J8.36 (Pin_36), R5.1
- new net: R8.2, U4.17 (~{RESET})
- no-connect marks 0 -> 255
Other:
- moved on the sheet: C1, C2, C3, C5, C6, C7, C8, IC1, J4, J5, J6, J7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

Commit message: pcb changes
Connections:
- net at C15.2, C16.2, C17.2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: now also IC1.55 (VIN_(3.6_TO_5.5_VOLTS)); no longer IC1.52 (+5V)
Changed lines of the file:
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@@
 	)
 	(no_connect
-		(at 222.25 207.01)
-	)
-	(no_connect
 		(at 196.85 54.61)
 	)
@@
 	)
 	(no_connect
+		(at 217.17 207.01)
+	)
+	(no_connect
 		(at 242.57 95.25)
 	)
@@
 	(wire
 		(pts
-			(xy 34.29 199.39) (xy 217.17 199.39)
+			(xy 34.29 199.39) (xy 222.25 199.39)
 		)
 		(stroke
@@
 	(wire
 		(pts
+			(xy 222.25 199.39) (xy 222.25 207.01)
+		)
+		(stroke
+			(width 0)
+			(type default)
+		)
+	)
+	(wire
+		(pts
 			(xy 280.67 34.29) (xy 273.05 34.29)
 		)
@@
 		)
 		(stroke
-			(width 0)
-			(type default)
-		)
-	)
-	(wire
-		(pts
-			(xy 217.17 199.39) (xy 217.17 207.01)
-		)
-		(stroke
